File: Module1/KiCad/OpenLEDModule1.sch (KiCad schematic (older format))
At the start: 8 parts, among them P1 CONN_01X02, P2 CONN_01X02

Commit message: Several fixes to resolve review comments (thermal via connections, cooling pads, footprint, past and mask layers, resistors, holes, tracks)
Parts:
- D1, D2, D3, D4: footprint blinkgestalten:LED_NICHIA -> OpenLed:LED_OsramDURIS_E5_JDSTS2EM
Changed lines of the file:
@@
 LIBS:contrib
 LIBS:valves
+LIBS:OpenLedModule
 LIBS:OpenLEDModule1-cache
 EELAYER 25 0
@@
 encoding utf-8
 Sheet 1 1
-Title "LED Modul Prototyp 1"
-Date ""
-Rev "1.0"
+Title "OpenLedModule 1"
+Date "2017-04-29"
+Rev "1.1"
 Comp "blinkgestalten"
 Comment1 ""
@@
 F 0 "D2" H 6150 3950 50  0000 C CNN
 F 1 "LED" H 6150 3750 50  0000 C CNN
-F 2 "blinkgestalten:LED_NICHIA" H 6150 3850 50  0001 C CNN
+F 2 "OpenLed:LED_OsramDURIS_E5_JDSTS2EM" H 6150 3850 50  0001 C CNN
 F 3 "" H 6150 3850 50  0000 C CNN
 	1    6150 3850
@@
 F 0 "D3" H 5300 3950 50  0000 C CNN
 F 1 "LED" H 5300 3750 50  0000 C CNN
-F 2 "blinkgestalten:LED_NICHIA" H 5300 3850 50  0001 C CNN
+F 2 "OpenLed:LED_OsramDURIS_E5_JDSTS2EM" H 5300 3850 50  0001 C CNN
 F 3 "" H 5300 3850 50  0000 C CNN
 	1    5300 3850
@@
 F 0 "D4" H 4900 3950 50  0000 C CNN
 F 1 "LED" H 4900 3750 50  0000 C CNN
-F 2 "blinkgestalten:LED_NICHIA" H 4900 3850 50  0001 C CNN
+F 2 "OpenLed:LED_OsramDURIS_E5_JDSTS2EM" H 4900 3850 50  0001 C CNN
 F 3 "" H 4900 3850 50  0000 C CNN
 	1    4900 3850
@@
 F 0 "D1" H 6550 3950 50  0000 C CNN
 F 1 "LED" H 6550 3750 50  0000 C CNN
-F 2 "blinkgestalten:LED_NICHIA" H 6550 3850 50  0001 C CNN
+F 2 "OpenLed:LED_OsramDURIS_E5_JDSTS2EM" H 6550 3850 50  0001 C CNN
 F 3 "" H 6550 3850 50  0000 C CNN
 	1    6550 3850
@@
 	4750 3850 4750 4250
 $Comp
-L PWR_FLAG #FLG?
+L PWR_FLAG #FLG03
 U 1 1 58F37C89
 P 7600 3350
-F 0 "#FLG?" H 7600 3445 50  0001 C CNN
+F 0 "#FLG03" H 7600 3445 50  0001 C CNN
 F 1 "PWR_FLAG" H 7600 3530 50  0000 C CNN
 F 2 "" H 7600 3350 50  0000 C CNN
@@
 $EndComp
 $Comp
-L PWR_FLAG #FLG?
+L PWR_FLAG #FLG04
 U 1 1 58F37CBD
 P 7600 4450
-F 0 "#FLG?" H 7600 4545 50  0001 C CNN
+F 0 "#FLG04" H 7600 4545 50  0001 C CNN
 F 1 "PWR_FLAG" H 7600 4630 50  0000 C CNN
 F 2 "" H 7600 4450 50  0000 C CNN
